Commit message: Added swri demo versions of urdf

File: crs_support/urdf/swri_demo.urdf (robot description, URDF)
Before this commit: robot swri_demo, 2 links, 1 joints
Links:
- added link base_link, mass 4.0; collision mesh filename=package://crs_support/meshes/ur10e/collision/base.stl; visual mesh filename=package://crs_support/meshes/ur10e/visual/base.dae
- added link camera_link_optical
- added link ee_link, mass 0.1; collision box size=0.01 0.01 0.01
- added link eoat_link, mass 0.202; collision cylinder length=0.20 radius=0.02; visual cylinder length=0.20 radius=0.02
- added link forearm_link, mass 3.87; collision mesh filename=package://crs_support/meshes/ur10e/collision/forearm_multib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; visual mesh filename=package://crs_support/meshes/ur10e/visual/forearm.dae
- added link robot_stand, mass 0.1; collision box size=0.4318 0.4318 1.1; collision box size=0.889 0.889 0.7112
- added link shoulder_link, mass 7.778; collision mesh filename=package://crs_support/meshes/ur10e/collision/shoulder.stl; visual mesh filename=package://crs_support/meshes/ur10e/visual/shoulder.dae
- added link upper_arm_link, mass 12.93; collision mesh filename=package://crs_support/meshes/ur10e/collision/upper_arm_mult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; visual mesh filename=package://crs_support/meshes/ur10e/visual/upperarm.dae
- added link world
- added link wrist_1_link, mass 1.96; collision mesh filename=package://crs_support/meshes/ur10e/collision/wrist1.stl; visual mesh filename=package://crs_support/meshes/ur10e/visual/wrist1.dae
- added link wrist_2_link, mass 1.96; collision mesh filename=package://crs_support/meshes/ur10e/collision/wrist2.stl; visual mesh filename=package://crs_support/meshes/ur10e/visual/wrist2.dae
- added link wrist_3_link, mass 0.202; collision mesh filename=package://crs_support/meshes/ur10e/collision/wrist3.stl; visual mesh filename=package://crs_support/meshes/ur10e/visual/wrist3.dae
Joints:
- removed joint base_to_tool0
- added joint base_link-base_fixed_joint: type fixed, parent base, child base_link, origin xyz=0 0 0 rpy=0 0 0
- added joint camera_optical_joint: type fixed, parent wrist_3_link, child camera_link_optical, origin xyz=0 0 0 rpy=-1.571 0 -1.571
- added joint ee_fixed_joint: type fixed, parent wrist_3_link, child ee_link, origin xyz=0.0 0.0 0.0 rpy=0.0 -1.57079632679 1.57079632679
- added joint elbow_joint: type revolute, parent upper_arm_link, child forearm_link, origin xyz=-0.611971344601 0 0 rpy=3.14047492209 3.14117521433 3.14159104748, axis 0 0 1, limit lower=-2.6 upper=3.141592653589793 effort=150.0 velocity=3.14
- added joint robot_base_joint: type fixed, parent robot_stand, child base, origin xyz=0 0 1.0922 rpy=0 0 0, limit lower=-0.1 upper=1.9 effort=1.0 velocity=.01
- added joint robot_stand_joint: type fixed, parent world, child robot_stand, origin xyz=0 0 0 rpy=0 0 0
- added joint shoulder_lift_joint: type revolute, parent shoulder_link, child upper_arm_link, origin xyz=0.00013292041689 0 0 rpy=1.57065145242 0 -2.70337965131e-06, axis 0 0 1, limit lower=-6.28318530718 upper=6.28318530718 effort=330.0 velocity=3.14
- added joint shoulder_pan_joint: type revolute, parent base_link, child shoulder_link, origin xyz=0 0 0.180920744391 rpy=0 0 3.14159249728, axis 0 0 1, limit lower=-6.28318530718 upper=6.28318530718 effort=330.0 velocity=3.14
- added joint tool0_to_eoat_link: type fixed, parent tool0, child eoat_link, origin xyz=0.0 0.0 0.0 rpy=0.0 0.0 0.0
- added joint wrist_1_joint: type revolute, parent forearm_link, child wrist_1_link, origin xyz=-0.571064941288 0.000500820247035 0.174414995927 rpy=3.13872123266 -3.14053617519 3.14158723656, axis 0 0 1, limit lower=-6.28318530718 upper=6.28318530718 effort=54.0 velocity=6.28
- added joint wrist_2_joint: type revolute, parent wrist_1_link, child wrist_2_link, origin xyz=5.96404309737e-05 -0.119843553735 -4.54415414531e-05 rpy=1.57117550062 0 -9.13444434245e-07, axis 0 0 1, limit lower=-6.28318530718 upper=6.28318530718 effort=54.0 velocity=6.28
- added joint wrist_3_joint: type revolute, parent wrist_2_link, child wrist_3_link, origin xyz=1.57784168351e-05 0.115533666641 0.000104843358957 rpy=1.57170379674 3.14159265359 3.14159254819, axis 0 0 1, limit lower=-6.28318530718 upper=6.28318530718 effort=54.0 velocity=6.28
- added joint wrist_3_link-tool0_fixed_joint: type fixed, parent wrist_3_link, child tool0, origin xyz=0 0 0 rpy=0 0 0
