Commit message: Added self collisions and updated robot name

File: crs_support/urdf/crs.urdf (robot description, URDF)
Before this commit: robot crs2, 14 links, 13 joints
Joints:
- joint robot_base_joint: axis (none) -> 1 0 0; limit lower=-0.1 upper=1.9 effort=54.0 velocity=.1 -> lower=-0.1 upper=1.9 effort=1.0 velocity=.01

Commit message: Smaller meshes to load in RVIZ and updated urdf correspondingly

File: crs_support/urdf/crs.urdf (robot description, URDF)
Before this commit: robot crs, 14 links, 13 joints
Links:
- link eoat_link: mass 0.202 -> 0.01; geometry collision mesh filename=package://crs_support/meshes/end_effector/collision/FRAMOS_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; visual mesh filename=package://crs_support/meshes/end_effector/visual/FRAMOS.stl
Joints:
- joint tool0_to_eoat_link: origin xyz=0.0 0.0 0.0 rpy=0.0 0.0 0.0 -> xyz=-0.04 0.09 -0.03 rpy=1.57 0.0 0

File: crs_support/urdf/swri_demo.urdf (robot description, URDF)
Before this commit: robot crs, 14 links, 13 joints
Links:
- link eoat_link: mass 0.202 -> 0.01; geometry collision mesh filename=package://crs_support/meshes/end_effector/collision/FRAMOS_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; visual mesh filename=package://crs_support/meshes/end_effector/visual/FRAMOS.stl
Joints:
- joint tool0_to_eoat_link: origin xyz=0.0 0.0 0.0 rpy=0.0 0.0 0.0 -> xyz=-0.04 0.09 -0.03 rpy=1.57 0.0 0

Commit message: Updated FRAMOS optical frame

File: crs_support/urdf/crs.urdf (robot description, URDF)
Before this commit: robot crs, 14 links, 13 joints
Links:
- added link gazebo_camera_link
Joints:
- added joint gazebo_camera_joint: type fixed, parent wrist_3_link, child gazebo_camera_link, origin xyz=0 0 0.02 rpy=0 0 1.571
- joint camera_optical_joint: parent wrist_3_link -> gazebo_camera_link

File: crs_support/urdf/swri_demo.urdf (robot description, URDF)
Before this commit: robot crs, 14 links, 13 joints
Links:
- added link gazebo_camera_link
Joints:
- added joint gazebo_camera_joint: type fixed, parent wrist_3_link, child gazebo_camera_link, origin xyz=0 0 0.02 rpy=0 0 1.571
- joint camera_optical_joint: parent wrist_3_link -> gazebo_camera_link

Commit message: Added cart to main mockup urdf

File: crs_support/urdf/crs.urdf (robot description, URDF)
Before this commit: robot crs, 15 links, 14 joints
Links:
- link robot_stand: geometry collision box size=0.05 2.25 2.7; collision box size=0.05 2.25 2.7
