Commit message: Updated swri urdf envrionment

File: crs_support/urdf/swri_demo2.urdf.xacro (robot description, xacro)
@@ -2,4 +2,78 @@
 <robot name="crs" xmlns:xacro="http://ros.org/wiki/xacro">
   <xacro:macro name="crs_workcell" params="prefix:=^|''">
+  <xacro:arg name="table_size" default="1.5"/>
+  <xacro:property name="BASE_PLATE_THICKNESS" value="0.00635" scope="parent"/>
+  <xacro:property name="BASE_PLATE_LENGTH" value="0.762" scope="parent"/>
+  <xacro:property name="BASE_PLATE_WIDTH" value="0.3048" scope="parent"/>
+    <link name="table">
+      <visual>
+        <origin xyz="0 0 -0.05"/>
+        <geometry>
+          <box size="$(arg table_size) $(arg table_size) 0.1"/>
+        </geometry>
+        <material name="StainlessSteel">
+          <color rgba="0.8 0.8 0.8 0.9"/>
+        </material>
+      </visual>
+      <collision>
+        <origin xyz="0 0 -0.05"/>
+        <geometry>
+          <box size="$(arg table_size) $(arg table_size) 0.1"/>
+        </geometry>
+      </collision>
+    </link>
+    <joint name="world_to_table_joint" type="fixed">
+      <origin xyz="0 0 1.0"/>
+      <parent link="world"/>
+      <child link="table"/>
+    </joint>
+    <link name="base_plate">
+      <visual>
+        <origin xyz="${0.5 * BASE_PLATE_WIDTH} ${0.5 * BASE_PLATE_LENGTH} ${BASE_PLATE_THICKNESS}"/>
+        <geometry>
+          <box size="${BASE_PLATE_WIDTH} ${BASE_PLATE_LENGTH} ${BASE_PLATE_THICKNESS}"/>
+        </geometry>
+        <material name="StainlessSteel">
+          <color rgba="0.6 0.6 0.6 1.0"/>
+        </material>
+      </visual>
+      <collision>
+        <origin xyz="${0.5 * BASE_PLATE_WIDTH} ${0.5 * BASE_PLATE_LENGTH} ${BASE_PLATE_THICKNESS}"/>
+        <geometry>
+          <box size="${BASE_PLATE_WIDTH} ${BASE_PLATE_LENGTH} ${BASE_PLATE_THICKNESS}"/>
+        </geometry>
+        <material name="StainlessSteel">
+          <color rgba="0.6 0.6 0.6 1.0"/>
+        </material>
+      </collision>
+    </link>
+    <joint name="table_to_base_plate" type="fixed">
+      <origin xyz="${-0.5*$(arg table_size) + 0.1397 } ${-0.5*$(arg table_size) + 0.09525} 0.0" rpy="0 0 0"/>
+       <parent link="table"/>
+       <child link="base_plate"/>
+    </joint>
+    <!-- mold -->
+    <link name="layup_mold">
+      <visual>
+        <origin xyz="0 0 0" rpy="0 0 0"/>
+        <geometry>
+         <mesh filename="package://crs_support/meshes/Swri_demo/mold_transformed.stl"/>
+        </geometry>
+        <material name="white">
+          <color rgba="1 1 1 1"/>
+        </material>
+      </visual>
+      <collision>
+        <origin xyz="0 0 0"/>
+        <geometry>
+          <mesh filename="package://crs_support/meshes/Swri_demo/mold_transformed.stl"/>
+        </geometry>
+      </collision>
+    </link>
+    <joint name="table_to_mold" type="fixed">
+      <parent link="table"/>
+      <child link="layup_mold"/>
+      <origin xyz="-0.30359 -0.13389 0.05497" rpy="-0.0091 -0.013 0.0197"/>
+    </joint>
     <link name="${prefix}base_link">
         <visual>
@@ -234,22 +308,43 @@
     </joint>
     <link name="${prefix}eoat_link">
-        <visual>
-            <geometry>
-                <mesh filename="package://crs_support/meshes/end_effector/visual/full_ee_v4.stl" />
-            </geometry>
-            <material name="Orange">
-                <color rgba="1.0 0.4 0.0 1.0" />
-            </material>
-        </visual>
-        <collision>
-            <geometry>
-                <mesh filename="package://crs_support/meshes/end_effector/collision/full_ee_v4_collision.stl" />
-            </geometry>
-        </collision>
-        <inertial>
-            <mass value="0.01" />
-            <origin rpy="0 0 0" xyz="0.0 0.0 0.0" />
-            <inertia ixx="0.000526462289415" ixy="0.0" ixz="0.0" iyy="0.000526462289415" iyz="0.0" izz="0.000568125" />
-        </inertial>
+        <inertial>
+            <origin xyz="8.625E-08 -4.6583E-06 0.03145" rpy="0 0 0" />
+            <mass value="0.22652" />
+            <inertia ixx="0.00020005" ixy="-4.2442E-10" ixz="-2.9069E-10" iyy="0.00017832" iyz="-3.4402E-08" izz="0.00013478" />
+        </inertial>
+        <visual>
+            <origin xyz="0 0 0" rpy="0 0 0" />
+            <geometry>
+                <mesh filename="package://crs_support/meshes/Swri_demo/robotiq_2f_85_gripper_visualization/collision/robotiq_arg2f_base_link.stl" />
+<!--                <mesh filename="package://crs_support/meshes/Swri_demo/robotiq_2f_85_gripper_visualization/visual/robotiq_arg2f_85_base_link.dae" scale="0.001 0.001 0.001"/>-->
+            </geometry>
+            <material name="">
+                <color rgba="0.1 0.1 0.1 1" />
+            </material>
+        </visual>
+        <collision>
+            <origin xyz="0 0 0" rpy="0 0 0" />
+            <geometry>
+                <mesh filename="package://crs_support/meshes/Swri_demo/robotiq_2f_85_gripper_visualization/collision/robotiq_arg2f_base_link.stl" />
+            </geometry>
+        </collision>
+        <visual>
+            <geometry>
+                <cylinder radius="0.015" length="0.175"/>
+            </geometry>
+            <origin rpy="0 0 0" xyz="0 0 0.0875" />
+            <material name="">
+                <color rgba="0.1 0.1 0.1 1" />
+            </material>
+        </visual>
+        <collision>
+            <geometry>
+                <cylinder radius="0.015" length="0.175"/>
+            </geometry>
+            <origin rpy="0 0 0" xyz="0 0 0.0875" />
+            <material name="">
+                <color rgba="0.1 0.1 0.1 1" />
+            </material>
+        </collision>
     </link>
     <joint name="${prefix}tool0_to_eoat_link" type="fixed">
@@ -259,5 +354,5 @@
     </joint>
     <link name="${prefix}robot_stand">
-        <visual>
+<!--        <visual>
             <geometry>
                 <box size="0.4318 0.4318 1.1"/>
@@ -334,10 +429,13 @@
             <mass value="0.1" />
             <inertia ixx="0.03" iyy="0.03" izz="0.03" ixy="0.0" ixz="0.0" iyz="0.0" />
-        </inertial>
+        </inertial>-->
     </link>
     <joint name="${prefix}robot_base_joint" type="fixed">
-        <parent link="robot_stand" />
+        <!--<parent link="robot_stand" />
         <child link="base" />
-        <origin rpy="0 0 0" xyz="0 0 1.0922" />
+        <origin rpy="0 0 0" xyz="0 0 1.0922" />-->
+        <parent link="layup_mold" />
+        <child link="base" />
+        <origin xyz="0.9545 0.0144 0.0797" rpy="0.0 0.0 3.1415"/>
         <limit effort="1.0" lower="-0.1" upper="1.9" velocity=".01" />
     </joint>
@@ -363,5 +461,6 @@
     <link name="${prefix}sander_center_link" />
     <joint name="${prefix}sander_joint" type = "fixed">
-        <origin xyz="0.0 -0.15497 0.17503" rpy="0.7854 0.0 0.0"/>
+<!--        <origin xyz="0.0 -0.15497 0.17503" rpy="0.7854 0.0 0.0"/>-->
+        <origin xyz="0.0 0.0 0.175" rpy="0.0 0.0 0.0"/>
         <parent link="${prefix}eoat_link"/>
         <child link="${prefix}sander_center_link" />
@@ -394,6 +493,6 @@
     <joint name="${prefix}robot_stand_to_part_joint" type= "fixed">
 <!--        <origin xyz="-0.5 0.5 1.3" rpy= "1.571 -1.571 0"/>-->
-        <origin xyz="-0.25 0.5 1.15" rpy= "0.0 0.0 0"/>
-        <parent link="${prefix}robot_stand"/>
+        <origin xyz="0.15 -0.5 0.0" rpy= "0.0 0.0 0"/>
+        <parent link="table"/>
         <child link="${prefix}part"/>
     </joint>

Commit message: WIP: testing

File: crs_support/urdf/swri_demo2.urdf.xacro (robot description, xacro)
@@ -3,5 +3,5 @@
   <xacro:macro name="crs_workcell" params="prefix:=^|''">
   <xacro:arg name="table_size" default="1.5"/>
-  <xacro:property name="BASE_PLATE_THICKNESS" value="0.00635" scope="parent"/>
+  <xacro:property name="BASE_PLATE_THICKNESS" value="0.6096" scope="parent"/> CHANGED TO ACCOUNT FOR KUKA
   <xacro:property name="BASE_PLATE_LENGTH" value="0.762" scope="parent"/>
   <xacro:property name="BASE_PLATE_WIDTH" value="0.3048" scope="parent"/>
@@ -30,5 +30,5 @@
     <link name="base_plate">
       <visual>
-        <origin xyz="${0.5 * BASE_PLATE_WIDTH} ${0.5 * BASE_PLATE_LENGTH} ${BASE_PLATE_THICKNESS}"/>
+        <origin xyz="${0.5 * BASE_PLATE_WIDTH} ${0.5 * BASE_PLATE_LENGTH} ${BASE_PLATE_THICKNESS * 0.5}"/>
         <geometry>
           <box size="${BASE_PLATE_WIDTH} ${BASE_PLATE_LENGTH} ${BASE_PLATE_THICKNESS}"/>
@@ -38,6 +38,6 @@
         </material>
       </visual>
-      <collision>
-        <origin xyz="${0.5 * BASE_PLATE_WIDTH} ${0.5 * BASE_PLATE_LENGTH} ${BASE_PLATE_THICKNESS}"/>
+<!--      <collision>
+        <origin xyz="${0.5 * BASE_PLATE_WIDTH} ${0.5 * BASE_PLATE_LENGTH} ${BASE_PLATE_THICKNESS * 0.5}"/>
         <geometry>
           <box size="${BASE_PLATE_WIDTH} ${BASE_PLATE_LENGTH} ${BASE_PLATE_THICKNESS}"/>
@@ -46,5 +46,5 @@
           <color rgba="0.6 0.6 0.6 1.0"/>
         </material>
-      </collision>
+      </collision>-->
     </link>
     <joint name="table_to_base_plate" type="fixed">
@@ -75,4 +75,47 @@
       <child link="layup_mold"/>
       <origin xyz="-0.30359 -0.13389 0.05497" rpy="-0.0091 -0.013 0.0197"/>
+    </joint>
+    <link name="table_obstacles">
+      <visual> Small square base plate
+        <origin xyz="0.2286 -0.127 0.005" rpy="0 0 0"/>
+        <geometry>
+          <box size="0.254 0.254 0.01"/>
+        </geometry>
+      </visual>
+      <visual> Clamp
+        <origin xyz="0.6985 -0.4445 0.1397" rpy="0 0 0"/>
+        <geometry>
+          <box size="0.1651 0.1143 0.2794"/>
+        </geometry>
+      </visual>
+      <visual> Assembly stuff
+        <origin xyz="0.38735 -0.4445 0.0254" rpy="0 0 0"/>
+        <geometry>
+          <box size="0.7747 0.1143 0.0508"/>
+        </geometry>
+      </visual>
+      <collision> Small square base plate
+        <origin xyz="0.2286 -0.127 0.005" rpy="0 0 0"/>
+        <geometry>
+          <box size="0.254 0.254 0.01"/>
+        </geometry>
+      </collision>
+      <collision> Clamp
+        <origin xyz="0.6985 -0.4445 0.1397" rpy="0 0 0"/>
+        <geometry>
+          <box size="0.1651 0.1143 0.2794"/>
+        </geometry>
+      </collision>
+      <collision> Assembly stuff
+        <origin xyz="0.38735 -0.4445 0.0254" rpy="0 0 0"/>
+        <geometry>
+          <box size="0.7747 0.1143 0.0508"/>
+        </geometry>
+      </collision>
+    </link>
+    <joint name="table_to_table_obstacles" type="fixed">
+      <parent link="table"/>
+      <child link="table_obstacles"/>
+      <origin xyz="-0.30359 -0.13389 0" rpy="0 0 0"/>
     </joint>
     <link name="${prefix}base_link">
@@ -493,5 +536,5 @@
     <joint name="${prefix}robot_stand_to_part_joint" type= "fixed">
 <!--        <origin xyz="-0.5 0.5 1.3" rpy= "1.571 -1.571 0"/>-->
-        <origin xyz="0.15 -0.5 0.0" rpy= "0.0 0.0 0"/>
+        <origin xyz="0.25 -0.28 0.0" rpy= "0.0 0.0 1.571"/>
         <parent link="table"/>
         <child link="${prefix}part"/>

Commit message: Added support for testing surface execution action

File: crs_support/urdf/swri_demo2.urdf.xacro (robot description, xacro)
@@ -38,5 +38,5 @@
         </material>
       </visual>
-<!--      <collision>
+      <collision>
         <origin xyz="${0.5 * BASE_PLATE_WIDTH} ${0.5 * BASE_PLATE_LENGTH} ${BASE_PLATE_THICKNESS * 0.5}"/>
         <geometry>
@@ -46,5 +46,5 @@
           <color rgba="0.6 0.6 0.6 1.0"/>
         </material>
-      </collision>-->
+      </collision>
     </link>
     <joint name="table_to_base_plate" type="fixed">
