Commit message: Added new mockup and cart to urdf

File: crs_support/urdf/crs.urdf.xacro (robot description, xacro)
@@ -262,5 +262,5 @@
             <origin rpy="1.57079632679 0 0" xyz="0 0 -0.1168" />
             <geometry>
-                <mesh filename="package://crs_support/meshes/Mockup/visual/mockup_frame_v3.stl" />
+                <mesh filename="package://crs_support/meshes/Mockup/visual/Mockup3_6_Frame_noTools_small.stl" />
             </geometry>
             <material name="LightGrey">
@@ -271,5 +271,5 @@
             <origin rpy="1.57079632679 0 0" xyz="0 0 -0.1168" />
             <geometry>
-                <mesh filename="package://crs_support/meshes/Mockup/visual/mockup_cart_v3.stl" />
+                <mesh filename="package://crs_support/meshes/Mockup/visual/mockup_cart_v4.stl" />
             </geometry>
             <material name="LightGrey">
@@ -280,42 +280,42 @@
             <origin rpy="1.57079632679 0 0" xyz="0 0 -0.1168" />
             <geometry>
-                <mesh filename="package://crs_support/meshes/Mockup/collision/mockup_cart_collision_v3.stl" />
+                <mesh filename="package://crs_support/meshes/Mockup/collision/Mockup3_6_Cart_collision.stl" />
             </geometry>
         </collision>
         <collision> <!-- Right Wall-->
             <geometry>
-                <box size="1.02 2.14 0.1" />
-            </geometry>
-            <origin rpy="0 0 0" xyz="-0.42 -1.1 1.105" />
+                <box size="3.0 2.14 0.1" />
+            </geometry>
+            <origin rpy="0 0 0" xyz="-0.5 -1.1 1.38" />
         </collision>
         <collision> <!-- Left Wall-->
             <geometry>
-                <box size="1.02 2.14 0.1" />
-            </geometry>
-            <origin rpy="0 0 0" xyz="-0.42 -1.1 -1.46" />
+                <box size="3.0 2.14 0.1" />
+            </geometry>
+            <origin rpy="0 0 0" xyz="-0.5 -1.1 -1.33" />
         </collision>
         <collision> Front Wall
             <geometry>
-                <box size="0.1 2.14 2.65" />
-            </geometry>
-            <origin rpy="0 0 0" xyz="0.4 -1.1 -0.175" />
+                <box size="0.1 2.14 3.0" />
+            </geometry>
+            <origin rpy="0 0 0" xyz="0.85 -1.1 0.0" />
         </collision>
         <collision> Back Wall
             <geometry>
-                <box size="0.1 2.14 2.65" />
-            </geometry>
-            <origin rpy="0 0 0" xyz="-1.25 -1.1 -0.175" />
+                <box size="0.1 2.14 3.0" />
+            </geometry>
+            <origin rpy="0 0 0" xyz="-2.06 -1.1 0.0" />
         </collision>
         <collision> <!-- Top front beam-->
             <geometry>
-                <box size="0.22 0.12 2.65" />
-            </geometry>
-            <origin rpy="0 0 0" xyz="0.036983 -2.145 -0.175" />
+                <box size="1.25 0.12 3.0" />
+            </geometry>
+            <origin rpy="0 0 0" xyz="0.38 -2.135 0.0" />
         </collision>
         <collision> <!-- Top back beam-->
             <geometry>
-                <box size="0.22 0.12 2.65" />
-            </geometry>
-            <origin rpy="0 0 0" xyz="-0.867 -2.145 -0.175" />
+                <box size="1.25 0.12 3.0" />
+            </geometry>
+            <origin rpy="0 0 0" xyz="-1.56 -2.135 0.0" />
         </collision>
         <inertial>
@@ -327,5 +327,5 @@
         <parent link="${prefix}robot_stand" />
         <child link="${prefix}base" />
-        <origin rpy="0 1.571 0" xyz="0.036983 -2.0948 0.58 " />
+        <origin rpy="0 1.570796 0" xyz="-0.148896 -2.047406 0.6277 " />
         <axis xyz="1 0 0"/>
         <limit effort="1.0" lower="-0.1" upper="1.9" velocity=".01" />

Commit message: Added new sander end effector

File: crs_support/urdf/crs.urdf.xacro (robot description, xacro)
@@ -236,5 +236,5 @@
         <visual>
             <geometry>
-                <mesh filename="package://crs_support/meshes/end_effector/visual/ee_v2.stl" />
+                <mesh filename="package://crs_support/meshes/end_effector/visual/full_ee_v4.stl" />
             </geometry>
             <material name="Orange">
@@ -244,5 +244,5 @@
         <collision>
             <geometry>
-                <mesh filename="package://crs_support/meshes/end_effector/collision/ee_v2_collision_full.stl" />
+                <mesh filename="package://crs_support/meshes/end_effector/collision/full_ee_v4_collision.stl" />
             </geometry>
         </collision>
@@ -352,5 +352,5 @@
     <link name="${prefix}sander_center_link" />
     <joint name="${prefix}sander_joint" type = "fixed">
-        <origin xyz="0.0 -0.1167 0.12664" rpy="0.7854 0.0 0.0"/>
+        <origin xyz="0.0 -0.15497 0.17503" rpy="0.7854 0.0 0.0"/>
         <parent link="${prefix}eoat_link"/>
         <child link="${prefix}sander_center_link" />

Commit message: Changes for testing different part positions

File: crs_support/urdf/crs.urdf.xacro (robot description, xacro)
@@ -271,18 +271,20 @@
         </visual>
         <visual>
+<!--            <origin rpy="1.57079632679 0 0" xyz="0.20 0 -0.1168" />-->
+            <origin rpy="1.57079632679 0 0" xyz="0.0 0.35 -0.1168" />
+            <geometry>
+                <mesh filename="package://crs_support/meshes/Mockup/visual/mockup_cart_v4.stl" />
+            </geometry>
+            <material name="LightGrey">
+                <color rgba="0.7 0.7 0.7 1.0" />
+            </material>
+        </visual>
+<!--        <collision>
             <origin rpy="1.57079632679 0 0" xyz="0.20 0 -0.1168" />
-            <geometry>
-                <mesh filename="package://crs_support/meshes/Mockup/visual/mockup_cart_v4.stl" />
-            </geometry>
-            <material name="LightGrey">
-                <color rgba="0.7 0.7 0.7 1.0" />
-            </material>
-        </visual>
-        <collision>
-            <origin rpy="1.57079632679 0 0" xyz="0.20 0 -0.1168" />
+            <origin rpy="1.57079632679 0 0" xyz="0.00 0.35 -0.1168" />
             <geometry>
                 <mesh filename="package://crs_support/meshes/Mockup/collision/Mockup3_6_Cart_collision.stl" />
             </geometry>
-        </collision>
+        </collision>-->
         <collision> <!-- Right Wall-->
             <geometry>
@@ -357,10 +359,10 @@
             <origin rpy="0 0.785 0" xyz="-2.06 -2.135 1.38" />
         </collision>
-        <collision> <!-- fake floor -->
+<!--        <collision> fake floor
             <geometry>
                 <box size="3.0 0.12 3.0" />
             </geometry>
             <origin rpy="0 0 0" xyz="-0.65 -0.82 0" />
-        </collision>
+        </collision>-->
         <inertial>
             <mass value="0.1" />

Commit message: Updated eoat

File: crs_support/urdf/crs.urdf.xacro (robot description, xacro)
@@ -279,10 +279,10 @@
             </material>
         </visual>
-        <collision>
+        <!--<collision>
             <origin rpy="1.57079632679 0 0" xyz="0.20 0 -0.1168" />
             <geometry>
                 <mesh filename="package://crs_support/meshes/Mockup/collision/Mockup3_6_Cart_collision.stl" />
             </geometry>
-        </collision>
+        </collision>-->
         <collision> <!-- Right Wall-->
             <geometry>
@@ -357,10 +357,10 @@
             <origin rpy="0 0.785 0" xyz="-2.06 -2.135 1.38" />
         </collision>
-        <collision> <!-- fake floor -->
+        <!--<collision>  fake floor
             <geometry>
                 <box size="3.0 0.12 3.0" />
             </geometry>
             <origin rpy="0 0 0" xyz="-0.65 -0.82 0" />
-        </collision>
+        </collision>-->
         <inertial>
             <mass value="0.1" />
@@ -402,5 +402,6 @@
         <child link="${prefix}camera_link"/>
     </joint>
-    <link name="${prefix}sander_center_link" >
+    <link name="${prefix}sander_center_link" />
+    <link name="${prefix}sander_intermediate_link">
       <visual>
           <geometry>
@@ -415,21 +416,20 @@
           <origin rpy="0 0 0" xyz="0 0 0" />
       </collision>
-      <collision>
-          <geometry>
-              <cylinder length="0.03" radius="0.115" />
-          </geometry>
-          <origin rpy="0 0 0" xyz="0 0 -0.105" />
-      </collision>
-<!--      <collision>
-          <geometry>
-              <cylinder length="0.025" radius="0.135" />
-          </geometry>
-          <origin rpy="0 0 0" xyz="0 0 -0.035" />
-      </collision>-->
-    </link>
-    <joint name="${prefix}sander_joint" type = "fixed">
+    </link>
+    <joint name="${prefix}sander_intermediate_to_sander_center_link" type="fixed">
+      <parent link="${prefix}sander_intermediate_link" />
+      <child link="${prefix}sander_center_link" />
+    <!--        <origin xyz="0 0.16578 0.01902" rpy="-0.785 0 0" />-->
+    <!--        <origin xyz="0 0.162 0.015" rpy="-0.785 0 0" />-->
+    <!--        <origin xyz="0 0.04612 -0.03371" rpy="-2.355 0 0" />-->
+      <origin  xyz="0.0 0.0 0.0125" rpy="0.0 0.0 0.0"/>
+    </joint>
+    <joint name="${prefix}tool0_to_sander_intermediate_link" type="fixed">
+        <parent link="${prefix}eoat_link" />
+        <child link="${prefix}sander_intermediate_link" />
+    <!--        <origin xyz="0 0.16578 0.01902" rpy="-0.785 0 0" />-->
+    <!--        <origin xyz="0 0.162 0.015" rpy="-0.785 0 0" />-->
+    <!--        <origin xyz="0 0.04612 -0.03371" rpy="-2.355 0 0" />-->
         <origin xyz="0.0 -0.15497 0.17503" rpy="0.7854 0.0 0.0"/>
-        <parent link="${prefix}eoat_link"/>
-        <child link="${prefix}sander_center_link" />
     </joint>
 <!--    <link name="${prefix}part" >

Commit message: Updated crs xacro to be more accurate

File: crs_support/urdf/crs.urdf.xacro (robot description, xacro)
@@ -30,5 +30,5 @@
         <axis xyz="0 0 1" />
 <!--        <limit effort="330.0" lower="-6.28318530718" upper="6.28318530718" velocity="3.14" />-->
-        <limit effort="330.0" lower="-4" upper="2.28" velocity="3.14" />
+        <limit effort="330.0" lower="-4" upper="3.28" velocity="3.14" />
         <dynamics damping="0.0" friction="0.0" />
     </joint>
@@ -271,5 +271,5 @@
         </visual>
         <visual>
-            <origin rpy="1.57079632679 0 0" xyz="0.20 0 -0.1168" />
+            <origin rpy="1.57079632679 0 0" xyz="0.00 0 -0.1168" />
             <geometry>
                 <mesh filename="package://crs_support/meshes/Mockup/visual/mockup_cart_v4.stl" />

Commit message: code cleanup and minor motion planning tweaks

File: crs_support/urdf/crs.urdf.xacro (robot description, xacro)
@@ -29,5 +29,4 @@
         <origin rpy="0 0 3.14159249728" xyz="0 0 0.180920744391" />
         <axis xyz="0 0 1" />
-<!--        <limit effort="330.0" lower="-6.28318530718" upper="6.28318530718" velocity="3.14" />-->
         <limit effort="330.0" lower="-4" upper="3.28" velocity="3.14" />
         <dynamics damping="0.0" friction="0.0" />
@@ -224,5 +223,4 @@
     <link name="${prefix}base" />
     <joint name="${prefix}base_link-base_fixed_joint" type="fixed">
-        <!--<origin rpy="-1.571 0 0" xyz="0 0 0" />-->
         <origin rpy="0 0 0" xyz="0 0 0" />-->
         <parent link="${prefix}base" />
@@ -279,10 +277,10 @@
             </material>
         </visual>
-        <!--<collision>
+        <collision>
             <origin rpy="1.57079632679 0 0" xyz="0.20 0 -0.1168" />
             <geometry>
                 <mesh filename="package://crs_support/meshes/Mockup/collision/Mockup3_6_Cart_collision.stl" />
             </geometry>
-        </collision>-->
+        </collision>
         <collision> <!-- Right Wall-->
             <geometry>
@@ -303,10 +301,4 @@
             <origin rpy="0 0 0" xyz="0.85 -1.1 0.0" />
         </collision>
-        <!--<collision> Back Wall Full
-            <geometry>
-                <box size="0.1 2.14 3.0" />
-            </geometry>
-            <origin rpy="0 0 0" xyz="-2.06 -1.1 0.0" />
-        </collision>-->
         <collision> Back Wall bottom Half
             <geometry>
@@ -333,10 +325,4 @@
             <origin rpy="0.786 0 0" xyz="-2.06 -1.9 -1.15" />
         </collision>
-<!--        <collision> < Top front beam>
-            <geometry>
-                <box size="1.25 0.12 3.0" />
-            </geometry>
-            <origin rpy="0 0 0" xyz="0.38 -2.135 0.0" />
-        </collision>-->
         <collision> <!-- Top back beam-->
             <geometry>
@@ -357,10 +343,10 @@
             <origin rpy="0 0.785 0" xyz="-2.06 -2.135 1.38" />
         </collision>
-        <!--<collision>  fake floor
-            <geometry>
-                <box size="3.0 0.12 3.0" />
+        <collision>  fake floor
+            <geometry>
+                <box size="3.0 0.12 2.5" />
             </geometry>
             <origin rpy="0 0 0" xyz="-0.65 -0.82 0" />
-        </collision>-->
+        </collision>
         <inertial>
             <mass value="0.1" />
@@ -371,5 +357,4 @@
         <parent link="${prefix}robot_stand" />
         <child link="${prefix}base" />
-<!--        <origin rpy="-1.570796 1.570796 0" xyz="-0.148896 -2.047406 0.6277 " />-->
         <origin rpy="-1.570796 1.570796 0" xyz="-1.030659 -2.037406 0.7977 " />
         <axis xyz="1 0 0"/>
@@ -390,12 +375,10 @@
     <link name="${prefix}camera_link_optical" />
     <joint name="${prefix}camera_optical_joint" type="fixed">
-        <origin xyz="-0.00345 0.070793 0.077409" rpy="-0.7854 0 0"/>
+        <origin xyz="-0.021 0.0797 0.06525" rpy="-0.7854 0 0"/>
         <parent link="${prefix}eoat_link"/>
-        <!-- <parent link="${prefix}gazebo_camera_link"/> -->
         <child link="${prefix}camera_link_optical"/>
     </joint>
     <link name="${prefix}camera_link" />
     <joint name="${prefix}camera_link_joint" type="fixed">
-<!--        <origin xyz="0.001 0.015 0.0" rpy="-1.57 1.57 0"/>-->
         <origin xyz="0.0 0.0 0.0" rpy="1.57 -1.57 0"/>
         <parent link="${prefix}camera_link_optical"/>
@@ -420,7 +403,4 @@
       <parent link="${prefix}sander_intermediate_link" />
       <child link="${prefix}sander_center_link" />
-    <!--        <origin xyz="0 0.16578 0.01902" rpy="-0.785 0 0" />-->
-    <!--        <origin xyz="0 0.162 0.015" rpy="-0.785 0 0" />-->
-    <!--        <origin xyz="0 0.04612 -0.03371" rpy="-2.355 0 0" />-->
       <origin  xyz="0.0 0.0 0.0125" rpy="0.0 0.0 0.0"/>
     </joint>
@@ -428,30 +408,6 @@
         <parent link="${prefix}eoat_link" />
         <child link="${prefix}sander_intermediate_link" />
-    <!--        <origin xyz="0 0.16578 0.01902" rpy="-0.785 0 0" />-->
-    <!--        <origin xyz="0 0.162 0.015" rpy="-0.785 0 0" />-->
-    <!--        <origin xyz="0 0.04612 -0.03371" rpy="-2.355 0 0" />-->
         <origin xyz="0.0 -0.15497 0.17503" rpy="0.7854 0.0 0.0"/>
     </joint>
-<!--    <link name="${prefix}part" >
-        <visual>
-            <origin rpy="0 0 0" xyz="0 0 0" />
-            <geometry>
-                <mesh filename="package://crs_support/meshes/Parts/visual/part1_ch.stl" />
-            </geometry>
-            <material name="Green">
-                <color rgba="0.0 0.7 0.0 1.0" />
-            </material>
-        </visual>
-        <collision>
-            <geometry>
-                <mesh filename="package://crs_support/meshes/Parts/collision/part1_ch.stl" />
-            </geometry>
-        </collision>
-    </link>
-    <joint name="${prefix}robot_stand_to_part_joint" type= "fixed">
-        <origin xyz="-0.439 -1.1 -0.14" rpy= "-3.1416 0.0 -1.571"/>
-        <parent link="${prefix}robot_stand"/>
-        <child link="${prefix}part"/>
-    </joint>-->
     <transmission name="trans_shoulder_pan_joint">
         <type>transmission_interface/SimpleTransmission</type>
@@ -617,12 +573,4 @@
           <joint_name>${prefix}wrist_3_joint</joint_name>
         </plugin>
-        <!-- Replaced by the crs_gazebo_plugins_joint_pose_trajectory plugin which hosts an action server instead
-        <plugin name='gazebo_ros_joint_pose_trajectory' filename='libgazebo_ros_joint_pose_trajectory.so'>
-            <ros>
-              <namespace>/demo</namespace>
-              <argument>set_joint_trajectory:=set_trajectory_test</argument>
-            </ros>
-            <update_rate>20</update_rate>
-        </plugin> -->
         <plugin name='crs_gazebo_plugins_joint_pose_trajectory' filename='libcrs_gazebo_plugins_joint_pose_trajectory.so'>
             <ros>

File: crs_support/urdf/swri_demo.urdf.xacro (robot description, xacro)
@@ -322,5 +322,5 @@
           </geometry>
       </collision>
-<!--      <inertial>
+<!--      <inertial> Keep this here for testing with other sander end effector
         <origin xyz="8.625E-08 -4.6583E-06 0.03145" rpy="0 0 0" />
         <origin xyz="0 0 0" rpy="0 0 0" />
@@ -409,10 +409,8 @@
         <origin xyz="-0.021 0.0797 0.06525" rpy="-0.7854 0 0"/>
         <parent link="${prefix}eoat_link"/>
-        <!-- <parent link="${prefix}gazebo_camera_link"/> -->
         <child link="${prefix}camera_link_optical"/>
     </joint>
     <link name="${prefix}camera_link" />
     <joint name="${prefix}camera_link_joint" type="fixed">
-<!--        <origin xyz="0.001 0.015 0.0" rpy="-1.57 1.57 0"/>-->
         <origin xyz="0.00 0.0 0.003" rpy="1.57 -1.57 0.0"/>
         <parent link="${prefix}camera_link_optical"/>

Commit message: Updated base position to middle of rail

File: crs_support/urdf/crs.urdf.xacro (robot description, xacro)
@@ -314,10 +314,10 @@
             <origin rpy="0 0 0" xyz="-0.5 -1.1 1.38" />
         </collision>
-        <collision> <!-- Left Wall-->
+       <!-- <collision> Left Wall
             <geometry>
                 <box size="3.0 2.14 0.1" />
             </geometry>
             <origin rpy="0 0 0" xyz="-0.5 -1.1 -1.33" />
-        </collision>
+        </collision>-->
         <collision> Front Wall
             <geometry>
@@ -356,11 +356,11 @@
             <origin rpy="0 0 0" xyz="-1.0 -2.135 0.0" />
         </collision>
-        <collision> <!-- Corner Bracket 1-->
+        <!--<collision> Corner Bracket 1
             <geometry>
                 <box size="1.25 0.12 1.25" />
             </geometry>
             <origin rpy="0 0.785 0" xyz="-2.06 -2.135 -1.33" />
-        </collision>
-        <collision> <!-- Corner Bracket 2-->
+        </collision>-->
+        <collision> Corner Bracket 2
             <geometry>
                 <box size="1.25 0.12 1.25" />
@@ -382,5 +382,6 @@
         <parent link="${prefix}robot_stand" />
         <child link="${prefix}base" />
-        <origin rpy="-1.570796 -1.570796 0.0" xyz="-1.030659 -2.037406 0.7977 " />
+<!--        <origin rpy="-1.570796 -1.570796 0.0" xyz="-1.030659 -2.037406 0.7977 " />-->
+        <origin rpy="-1.570796 -1.570796 0.0" xyz="-1.030659 -2.037406 0.2 " />
         <axis xyz="1 0 0"/>
         <limit effort="1.0" lower="-0.1" upper="1.9" velocity=".01" />
