Commit message: improved trajopt results

File: crs_support/urdf/swri_demo.urdf.xacro (robot description, xacro)
@@ -14,10 +14,10 @@
         </material>
       </visual>
-      <collision>
+<!--      <collision>
         <origin xyz="0 0 -0.05"/>
         <geometry>
           <box size="$(arg table_size) $(arg table_size) 0.1"/>
         </geometry>
-      </collision>
+      </collision>-->
     </link>
     <joint name="world_to_table_joint" type="fixed">

Commit message: removed wall to test swri part

File: crs_support/urdf/swri_demo.urdf.xacro (robot description, xacro)
@@ -54,5 +54,5 @@
     </joint>
     <link name="${prefix}external_walls">
-      <visual>
+      <!--<visual>
         <origin xyz="0 0.765 0"/>
         <geometry>
@@ -65,5 +65,5 @@
           <box size="$(arg table_size) 0.1 $(arg table_size)"/>
         </geometry>
-      </collision>
+      </collision>-->
     </link>
     <joint name="table_to_external_walls" type="fixed">

Commit message: updated camera position

File: crs_support/urdf/swri_demo.urdf.xacro (robot description, xacro)
@@ -14,10 +14,10 @@
         </material>
       </visual>
-<!--      <collision>
+      <collision>
         <origin xyz="0 0 -0.05"/>
         <geometry>
           <box size="$(arg table_size) $(arg table_size) 0.1"/>
         </geometry>
-      </collision>-->
+      </collision>
     </link>
     <joint name="world_to_table_joint" type="fixed">
@@ -407,5 +407,5 @@
     <link name="${prefix}camera_link_optical" />
     <joint name="${prefix}camera_optical_joint" type="fixed">
-        <origin xyz="-0.00345 0.070793 0.077409" rpy="-0.7854 0 0"/>
+        <origin xyz="-0.021 0.0797 0.06525" rpy="-0.7854 0 0"/>
         <parent link="${prefix}eoat_link"/>
         <!-- <parent link="${prefix}gazebo_camera_link"/> -->
@@ -415,5 +415,5 @@
     <joint name="${prefix}camera_link_joint" type="fixed">
 <!--        <origin xyz="0.001 0.015 0.0" rpy="-1.57 1.57 0"/>-->
-        <origin xyz="0.0 0.0 0.0" rpy="1.57 -1.57 0"/>
+        <origin xyz="0.00 0.0 0.003" rpy="1.57 -1.57 0.0"/>
         <parent link="${prefix}camera_link_optical"/>
         <child link="${prefix}camera_link"/>

Commit message: Updated sander frame for alternate EE

File: crs_support/urdf/swri_demo.urdf.xacro (robot description, xacro)
@@ -66,4 +66,28 @@
         </geometry>
       </collision>-->
+      <visual>
+        <origin xyz="0.61 -0.7 -0.33"/>
+        <geometry>
+          <box size="0.15 0.15 1.0"/>
+        </geometry>
+      </visual>
+      <collision>
+        <origin xyz="0.61 -0.7 -0.33"/>
+        <geometry>
+          <box size="0.15 0.15 1.0"/>
+        </geometry>
+      </collision>
+      <visual>
+        <origin xyz="-0.55 -0.7 -0.33"/>
+        <geometry>
+          <box size="0.15 0.15 1.0"/>
+        </geometry>
+      </visual>
+      <collision>
+        <origin xyz="-0.55 -0.7 -0.33"/>
+        <geometry>
+          <box size="0.15 0.15 1.0"/>
+        </geometry>
+      </collision>
     </link>
     <joint name="table_to_external_walls" type="fixed">
@@ -389,5 +413,5 @@
 <!--        <origin xyz="0 0.162 0.015" rpy="-0.785 0 0" />-->
 <!--        <origin xyz="0 0.04612 -0.03371" rpy="-2.355 0 0" />-->
-      <origin  xyz="0.0 0.0 0.0125" rpy="0.0 0.0 0.0"/>
+      <origin  xyz="0.0 0.0 0.00" rpy="0.0 0.0 0.0"/>
     </joint>
     <joint name="${prefix}tool0_to_sander_intermediate_link" type="fixed">

Commit message: Local uncommited changes

File: crs_support/urdf/swri_demo.urdf.xacro (robot description, xacro)
@@ -4,6 +4,6 @@
   <xacro:arg name="table_size" default="3.0"/>
     <link name="world"/>
-    <link name="table">
-      <visual>
+    <link name="${prefix}table">
+      <!--<visual>
         <origin xyz="0 0 -0.05"/>
         <geometry>
@@ -19,10 +19,10 @@
           <box size="$(arg table_size) $(arg table_size) 0.1"/>
         </geometry>
-      </collision>
+      </collision>-->
     </link>
     <joint name="world_to_table_joint" type="fixed">
       <origin xyz="0 0 ${-0.353 - 0.010}"/>
       <parent link="world"/>
-      <child link="table"/>
+      <child link="${prefix}table"/>
     </joint>
   <!--  <link name="${prefix}part"/>
@@ -32,5 +32,5 @@
       <child link="${prefix}part"/>
     </joint>-->
-    <link name="robot_stand">
+    <link name="${prefix}robot_stand">
       <visual>
         <origin xyz="0 0 -0.1905"/>
@@ -49,5 +49,5 @@
       <origin xyz="0.0 0.0 0.0" rpy="0.0 0.0 3.1415"/>
       <parent link="world"/>
-      <child link="robot_stand"/>
+      <child link="${prefix}robot_stand"/>
     </joint>
     <link name="${prefix}external_walls">
@@ -182,4 +182,17 @@
         </inertial>
     </link>
+    <joint name="${prefix}wrist_protective_stop_guard_joint" type="fixed">
+      <parent link="${prefix}forearm_link"/>
+      <child link="${prefix}wrist_protective_stop_guard_link"/>
+      <origin rpy="0 0 0" xyz="0 0 0"/>
+    </joint>
+    <link name="${prefix}wrist_protective_stop_guard_link">
+      <collision>
+        <origin rpy="1.57079632679 0 -1.57079632679" xyz="0.0 0.0 0.0393"/>
+        <geometry>
+          <mesh filename="package://crs_support/meshes/ur10e/collision/wrist_protective_stop_guard.stl"/>
+        </geometry>
+      </collision>
+    </link>
     <joint name="${prefix}wrist_1_joint" type="revolute">
         <parent link="${prefix}forearm_link" />
@@ -290,7 +303,7 @@
     </link>
     <link name="${prefix}base" />
-    <joint name="table_to_ur" type="fixed">
-      <origin xyz="0.0 0.0 0.0" rpy="0.0 0.0 3.1415"/>
-      <parent link="world"/>
+    <joint name="${prefix}robot_base_joint" type="fixed">
+      <origin xyz="0.0 0.0 0.0" rpy="0.0 0.0 0.0"/>
+      <parent link="${prefix}robot_stand"/>
       <child link="${prefix}base"/>
     </joint>
@@ -358,4 +371,53 @@
     <link name="${prefix}sander_center_link" />
     <link name="${prefix}sander_intermediate_link">
+      <!--<visual>
+          <geometry>
+              <cylinder length="0.06" radius="0.06425" />
+          </geometry>
+          <origin rpy="0 0 0" xyz="0 0 0" />
+      </visual>
+      <collision>
+          <geometry>
+              <cylinder length="0.025" radius="0.06425" />
+          </geometry>
+          <origin rpy="0 0 0" xyz="0 0 0" />
+      </collision>
+      <visual>
+          <geometry>
+              <cylinder length="0.20" radius="0.0125" />
+          </geometry>
+          <origin rpy="1.57 0 0" xyz="-0.0175 -0.1 -.0375" />
+      </visual>
+      <visual>
+          <geometry>
+              <cylinder length="0.0254" radius="0.0125" />
+          </geometry>
+          <origin rpy="0 1.57 0" xyz="0.0 -0.2 -.0375" />
+      </visual>
+      <collision>
+          <geometry>
+              <cylinder length="0.20" radius="0.0125" />
+          </geometry>
+          <origin rpy="1.57 0 0" xyz="-0.0175 -0.1 -.0375" />
+      </collision>
+      <collision>
+          <geometry>
+              <cylinder length="0.0254" radius="0.0125" />
+          </geometry>
+          <origin rpy="0 1.57 0" xyz="0.0 -0.2 -.0375" />
+      </collision>-->
+    </link>
+    <joint name="${prefix}sander_intermediate_to_sander_center_link" type="fixed">
+      <parent link="${prefix}sander_intermediate_link" />
+      <child link="${prefix}sander_center_link" />
+      <origin  xyz="0.0 0.0 0.00" rpy="0.0 0.0 0.0"/>
+    </joint>
+    <joint name="${prefix}tool0_to_sander_intermediate_link" type="fixed">
+        <parent link="${prefix}eoat_link" />
+        <child link="${prefix}sander_intermediate_link" />
+        <origin xyz="0.0 -0.17503 0.15497" rpy="0.7854 0.0 0.0"/>
+    </joint>
+    <!--<link name="${prefix}sander_center_link" />
+    <link name="${prefix}sander_intermediate_link">
       <visual>
           <geometry>
@@ -380,5 +442,5 @@
         <child link="${prefix}sander_intermediate_link" />
         <origin xyz="0.0 -0.15497 0.17503" rpy="0.7854 0.0 0.0"/>
-    </joint>
+    </joint>-->
     <link name="${prefix}gazebo_camera_link" />
     <joint name="${prefix}gazebo_camera_joint" type="fixed">
@@ -396,5 +458,5 @@
     <link name="${prefix}camera_link" />
     <joint name="${prefix}camera_link_joint" type="fixed">
-        <origin xyz="0.00 0.0 0.003" rpy="1.57 -1.57 0.0"/>
+        <origin xyz="0.00 0.0 -0.005" rpy="1.57 -1.57 0.0"/>
         <parent link="${prefix}camera_link_optical"/>
         <child link="${prefix}camera_link"/>
